File: EPS PCB/EPS_PCB_PrototypingV2/curr_meas.kicad_sch (KiCad schematic)
At the start: 36 parts, among them Q1 DMG6968U, Q2 DMG6968U, Q3 2N7002, Q4 2N7002, Q5 DMG6968U, Q6 2N7002, U6 STEF033APUR, U7 STEF512PUR, U8 INA3221

Commit message: EPS PCB Ready for Order
Parts:
- renumbered R20 to R19, R19 to R20
Connections:
- net 3V3_out: no longer C20.1, C22.1, R14.1, R15.1, R16.1, R17.1, R18.1, R19.1, U8.16 (VPU)
- net 5V_HK: now also C20.1, C22.1, R14.1, R15.1, R16.1, R17.1, R18.1, R19.1, U8.16 (VPU)
