File: EPS PCB/EPS_PCB_PrototypingV2/watchdog_timer.kicad_sch (KiCad schematic)
At the start: 6 parts, among them J8 Conn_01x02_Pin, U5 TPS3431SDRBR

Commit message: EPS PCB Ready for Order
Parts:
- renumbered J8 to J9
