File: EPS PCB/EPS_PCB_PrototypingV2/EPS_PCB_Prototyping.kicad_pcb (KiCad board)
At the start: 2 copper layers, 95.9 x 90.2 mm, 91 parts, among them J1 Conn_02x26_Row_Letter_First, J2 Conn_02x26_Row_Letter_First, J3 Conn_01x02_Pin, J4 Conn_01x02_Pin, J5 Conn_01x02_Pin, J6 Conn_01x02_Pin, J8 Conn_01x02_Pin, Q1 DMG6968U, Q2 DMG6968U, Q3 2N7002, Q4 2N7002, Q5 DMG6968U, Q6 2N7002, U1 TPS5430DDA, U2 TPS5430DDA, U3 TPS5430DDA, U4 TPS7A1650DGNR, U5 TPS3431SDRBR, U6 STEF033APUR, U7 STEF512PUR, U8 INA3221, U9 TLV3691IDPFR

Commit message: EPS PCB Ready for Order
Parts:
- added G***: LOGO, LOGO, F.Cu at (152.8, 57.5)
- added J3: Conn_01x08_Pin, Connector_PinHeader_2.54mm:PinHeader_1x08_P2.54mm_Vertical, F.Cu at (175.2, 54.4)
- added J4: Conn_01x06_Pin, Connector_PinHeader_2.54mm:PinHeader_1x06_P2.54mm_Horizontal, F.Cu at (190.6, 125.4)
- H1, H2, H3, H4: footprint MountingHole:MountingHole_3.2mm_M3_Pad_TopBottom -> MountingHole:MountingHole_3.2mm_M3_Pad
- U7: footprint Footprints:STEF512 -> Footprints:QFN10_2X3_STM-L
- moved L2 0.32 mm to (210.4, 89.5)
- renumbered J3 to J5, J4 to J6, J5 to J7, J6 to J8, J8 to J9, R20 to R19, R19 to R20
Connections:
- C20 pad 1: 3V3_out -> 5V_HK
- C22 pad 1: 3V3_out -> 5V_HK
- J1 pad a1: GND -> unconnected-(J1-Pin_a1-Pada1)
- J1 pad a10: unconnected-(J1-Pin_a10-Pada10) -> ACDS_PWM_2
- J1 pad a11: 12V_en -> ACDS_PWM_3
- J1 pad a12: 12V_out -> ACDS_PWM_4
- J1 pad a13: unconnected-(J1-Pin_a13-Pada13) -> 5V_out
- J1 pad a15: CM_SCL -> ACDS_PERM_5
- J1 pad a16: CM_SDA -> ACDS_PERM_6
- J1 pad a17: unconnected-(J1-Pin_a17-Pada17) -> GND
- J1 pad a20: unconnected-(J1-Pin_a20-Pada20) -> RS SYS2 Rx
- J1 pad a22: 3V3_en -> unconnected-(J1-Pin_a22-Pada22)
- J1 pad a23: 3V3_out -> unconnected-(J1-Pin_a23-Pada23)
- J1 pad a25: GPIO -> unconnected-(J1-Pin_a25-Pada25)
- J1 pad a26: GND -> unconnected-(J1-Pin_a26-Pada26)
- J1 pad a5: unconnected-(J1-Pin_a5-Pada5) -> STAT_2
- J1 pad a6: 5V_en -> unconnected-(J1-Pin_a6-Pada6)
- J1 pad a7: 5V_out -> unconnected-(J1-Pin_a7-Pada7)
- J1 pad a9: unconnected-(J1-Pin_a9-Pada9) -> ACDS_PWM_1
- J1 pad b1: GND -> unconnected-(J1-Pin_b1-Padb1)
- J1 pad b11: 12V_conv_out -> RS-485 SYS1 B
- J1 pad b12: 12V_out -> RS-485 SYS1 B
- J1 pad b13: unconnected-(J1-Pin_b13-Padb13) -> 5V_out
- J1 pad b14: WARNING -> unconnected-(J1-Pin_b14-Padb14)
- J1 pad b15: CRITICAL -> ACDS_IMU_RST
- J1 pad b16: PV -> unconnected-(J1-Pin_b16-Padb16)
- J1 pad b17: unconnected-(J1-Pin_b17-Padb17) -> GND
- J1 pad b20: unconnected-(J1-Pin_b20-Padb20) -> RS SYS2 Tx
- J1 pad b21: unconnected-(J1-Pin_b21-Padb21) -> UART_RX
- J1 pad b22: 3V3_conv_out -> UART_TX
- J1 pad b23: 3V3_out -> unconnected-(J1-Pin_b23-Padb23)
- J1 pad b25: RESET -> unconnected-(J1-Pin_b25-Padb25)
- J1 pad b26: GND -> unconnected-(J1-Pin_b26-Padb26)
- J1 pad b3: unconnected-(J1-Pin_b3-Padb3) -> ACDS_RS232_TX
- J1 pad b4: unconnected-(J1-Pin_b4-Padb4) -> ACDS_RS232_RX
- J1 pad b5: unconnected-(J1-Pin_b5-Padb5) -> PG
- J1 pad b6: 5V_conv_out -> INT
- J1 pad b7: 5V_out -> STAT_1
- J1 pad b8: unconnected-(J1-Pin_b8-Padb8) -> CM_SDA
- J1 pad b9: unconnected-(J1-Pin_b9-Padb9) -> CM_SCL
- J2 pad a1: unconnected-(J2-Pin_a1-Pada1) -> SUN_SENSE_1
- J2 pad a12: unconnected-(J2-Pin_a12-Pada12) -> 12V_out
- J2 pad a13: unconnected-(J2-Pin_a13-Pada13) -> 5V_out
- J2 pad a14: unconnected-(J2-Pin_a14-Pada14) -> 3V3_out
- J2 pad a2: unconnected-(J2-Pin_a2-Pada2) -> SUN_SENSE_3
- J2 pad a22: unconnected-(J2-Pin_a22-Pada22) -> SOL_PIN
- J2 pad a24: unconnected-(J2-Pin_a24-Pada24) -> V_Batt
- J2 pad a25: GND -> RBF_A
- J2 pad a26: GND -> DS_A
- J2 pad a3: unconnected-(J2-Pin_a3-Pada3) -> THR_1
- J2 pad a4: unconnected-(J2-Pin_a4-Pada4) -> THR_3
- J2 pad b1: unconnected-(J2-Pin_b1-Padb1) -> SUN_SENSE_2
- J2 pad b10: unconnected-(J2-Pin_b10-Padb10) -> HEATER_PWM
- J2 pad b12: unconnected-(J2-Pin_b12-Padb12) -> 12V_out
- J2 pad b13: unconnected-(J2-Pin_b13-Padb13) -> 5V_out
- J2 pad b14: unconnected-(J2-Pin_b14-Padb14) -> 3V3_out
- J2 pad b2: unconnected-(J2-Pin_b2-Padb2) -> SUN_SENSE_4
- J2 pad b22: unconnected-(J2-Pin_b22-Padb22) -> SOL_PIN
- J2 pad b23: V_Batt -> SYS_PIN
- J2 pad b24: unconnected-(J2-Pin_b24-Padb24) -> SYS_PIN
- J2 pad b25: GND -> RBF_B
- J2 pad b26: GND -> DS_B
- J2 pad b3: unconnected-(J2-Pin_b3-Padb3) -> THR_2
- J2 pad b4: unconnected-(J2-Pin_b4-Padb4) -> THR_4
- J2 pad b5: unconnected-(J2-Pin_b5-Padb5) -> THR_5
- J2 pad b6: unconnected-(J2-Pin_b6-Padb6) -> THR_6
- J2 pad b7: unconnected-(J2-Pin_b7-Padb7) -> THR_7
- J2 pad b8: unconnected-(J2-Pin_b8-Padb8) -> THR_8
- J2 pad b9: unconnected-(J2-Pin_b9-Padb9) -> THR_9
- R14 pad 1: 3V3_out -> 5V_HK
- R15 pad 1: 3V3_out -> 5V_HK
- R16 pad 1: 3V3_out -> 5V_HK
- R17 pad 1: 3V3_out -> 5V_HK
- R18 pad 1: 3V3_out -> 5V_HK
- R19 pad 1: 3V3_out -> 5V_HK
- U8 pad 16: 3V3_out -> 5V_HK
Routing:
- net 3V3_en: track 10.1 -> 129.6 mm, vias 0 -> 3
- net 5V_HK: track 180.6 -> 273.5 mm, vias 4 -> 10
- net 3V3_conv_out: track 58.4 -> 115.3 mm, vias 1 -> 3
- net 12V_en: track 8.34 -> 49.5 mm, vias 0 -> 1
- net RESET: track 93.8 -> 57.9 mm
- net 5V_en: track 7.71 -> 43.2 mm, vias 0 -> 1
- net 5V_conv_out: track 43.2 -> 10.8 mm, vias 1 -> 0
- net GPIO: track 86.0 -> 55.2 mm
- net 12V_out: track 0.86 -> 30.4 mm, vias 0 -> 2
- net 12V_conv_out: track 49.2 -> 26.9 mm, vias 1 -> 2
- net 3V3_out: track 76.6 -> 54.7 mm, vias 3 -> 1
- net CM_SCL: track 52.1 -> 72.4 mm
- net PV: track 68.2 -> 48.6 mm, vias 1 -> 2
- net CRITICAL: track 63.7 -> 45.0 mm, vias 1 -> 2
- net CM_SDA: track 52.3 -> 69.4 mm
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- added copper zone on B.Cu, net 12V_out
- removed copper zone on F.Cu, net 12V_out
Other:
- rule pad_to_mask_clearance: 0.051 -> 0

Commit message: Small PC104 Template Fix
Connections:
- J1 pad b12: RS-485 SYS1 B -> RS-485 SYS1 A
- U4 pad PAD: GND -> (no net)
- U4 pad V: GND -> (no net)
- U5 pad 10: GND -> (no net)
- U5 pad 11: GND -> (no net)
- U5 pad 12: GND -> (no net)
- U5 pad 13: GND -> (no net)
Routing:
- net RS-485 SYS1 B: track 2.54 -> 0.00 mm

Commit message: PDS Ordered
Parts:
- added J10: Conn_01x02_Pin, Connector_PinSocket_2.54mm:PinSocket_1x02_P2.54mm_Vertical, F.Cu at (215.7, 67.0)
- added J11: Conn_01x02_Pin, Connector_PinSocket_2.54mm:PinSocket_1x02_P2.54mm_Vertical, F.Cu at (215.4, 96.3)
- added J12: Conn_01x02_Pin, Connector_PinSocket_2.54mm:PinSocket_1x02_P2.54mm_Vertical, F.Cu at (210.4, 132.2)
- added J13: Conn_01x02_Pin, Connector_PinSocket_2.54mm:PinSocket_1x02_P2.54mm_Vertical, F.Cu at (189.4, 65.5)
- added J14: Conn_01x02_Pin, Connector_PinSocket_2.54mm:PinSocket_1x02_P2.54mm_Vertical, F.Cu at (189.7, 75.7)
- added J15: Conn_01x02_Pin, Connector_PinSocket_2.54mm:PinSocket_1x02_P2.54mm_Vertical, F.Cu at (192.9, 118.5)
- Q1, Q2, Q5: value DMG6968U -> DMG2305UX
- moved C15 0.77 mm to (191.9, 113.4)
- moved L2 0.45 mm to (209.9, 89.5)
Connections:
- C1 pad 1: V_Batt -> Net-(J10-Pin_2)
- C16 pad 1: 5V_conv_out -> Net-(J13-Pin_2)
- C19 pad 1: 3V3_conv_out -> Net-(J15-Pin_2)
- C2 pad 1: V_Batt -> Net-(J11-Pin_2)
- C26 pad 1: 12V_conv_out -> Net-(J14-Pin_1)
- C3 pad 1: V_Batt -> Net-(J12-Pin_2)
- U1 pad 7: V_Batt -> Net-(J10-Pin_2)
- U2 pad 7: V_Batt -> Net-(J11-Pin_2)
- U3 pad 7: V_Batt -> Net-(J12-Pin_2)
- U6 pad 11: 3V3_conv_out -> Net-(J15-Pin_2)
- U7 pad 10: 12V_conv_out -> Net-(J14-Pin_1)
- U7 pad 4: 5V_conv_out -> Net-(J13-Pin_2)
Routing:
- net V_Batt: track 217.5 -> 169.4 mm, vias 9 -> 7
- net Net-(J10-Pin_2): track 0.00 -> 16.1 mm, vias 0 -> 1
- net GND: track 158.1 -> 171.8 mm, vias 36 -> 47
- net Net-(J11-Pin_2): track 0.00 -> 12.3 mm
- net Net-(J12-Pin_2): track 0.00 -> 9.71 mm
- net Net-(J15-Pin_2): track 0.00 -> 8.03 mm
- net 3V3_conv_out: track 115.3 -> 111.2 mm, vias 3 -> 1
- net 12V_conv_out: track 26.9 -> 29.1 mm
- net 5V_conv_out: track 10.8 -> 8.78 mm
- net Net-(J13-Pin_2): track 0.00 -> 2.06 mm
- net Net-(J14-Pin_1): track 0.00 -> 1.99 mm
- net 5V_HK: track 273.5 -> 274.3 mm
- added copper zone on F.Cu, net Net-(J13-Pin_2)
- added copper zone on F.Cu, net Net-(J14-Pin_1)
