File: PCI-104-Temp/PCI-104-Librecube/PCI-104-Temp/PCI-104-Temp.kicad_pcb (KiCad board)
At the start: 2 copper layers, 95.9 x 90.2 mm, 6 parts, among them J3 Conn_02x26_Row_Letter_First, J4 Conn_02x26_Row_Letter_First

Commit message: EPS PCB Ready for Order
Parts:
- H1, H2, H3, H4: footprint MountingHole:MountingHole_3.2mm_M3_Pad_TopBottom -> MountingHole:MountingHole_3.2mm_M3_Pad
Connections:
- J3 pad a10: unconnected-(J3-Pin_a10-Pada10) -> ACDS_PWM_2
- J3 pad a11: unconnected-(J3-Pin_a11-Pada11) -> ACDS_PWM_3
- J3 pad a12: unconnected-(J3-Pin_a12-Pada12) -> ACDS_PWM_4
- J3 pad a13: unconnected-(J3-Pin_a13-Pada13) -> 5V_PERM
- J3 pad a15: unconnected-(J3-Pin_a15-Pada15) -> ACDS_PERM_5
- J3 pad a16: unconnected-(J3-Pin_a16-Pada16) -> ACDS_PERM_6
- J3 pad a17: unconnected-(J3-Pin_a17-Pada17) -> GND
- J3 pad a20: unconnected-(J3-Pin_a20-Pada20) -> RS SYS2 Rx
- J3 pad a26: GND -> unconnected-(J3-Pin_a26-Pada26)
- J3 pad a5: unconnected-(J3-Pin_a5-Pada5) -> STAT_2
- J3 pad a9: unconnected-(J3-Pin_a9-Pada9) -> ACDS_PWM_1
- J3 pad b11: unconnected-(J3-Pin_b11-Padb11) -> RS-485 SYS1 B
- J3 pad b12: unconnected-(J3-Pin_b12-Padb12) -> RS-485 SYS1 B
- J3 pad b13: unconnected-(J3-Pin_b13-Padb13) -> 5V_PERM
- J3 pad b15: unconnected-(J3-Pin_b15-Padb15) -> ACDS_IMU_RST
- J3 pad b17: unconnected-(J3-Pin_b17-Padb17) -> GND
- J3 pad b20: unconnected-(J3-Pin_b20-Padb20) -> RS SYS2 Tx
- J3 pad b21: unconnected-(J3-Pin_b21-Padb21) -> UART_RX
- J3 pad b22: unconnected-(J3-Pin_b22-Padb22) -> UART_TX
- J3 pad b26: GND -> unconnected-(J3-Pin_b26-Padb26)
- J3 pad b3: unconnected-(J3-Pin_b3-Padb3) -> ACDS_RS232_TX
- J3 pad b4: unconnected-(J3-Pin_b4-Padb4) -> ACDS_RS232_RX
- J3 pad b5: unconnected-(J3-Pin_b5-Padb5) -> PG
- J3 pad b6: unconnected-(J3-Pin_b6-Padb6) -> INT
- J3 pad b7: unconnected-(J3-Pin_b7-Padb7) -> STAT_1
- J3 pad b8: unconnected-(J3-Pin_b8-Padb8) -> SDA
- J3 pad b9: unconnected-(J3-Pin_b9-Padb9) -> SCL
- J4 pad a1: unconnected-(J4-Pin_a1-Pada1) -> SUN_SENSE_1
- J4 pad a12: unconnected-(J4-Pin_a12-Pada12) -> 12V
- J4 pad a13: unconnected-(J4-Pin_a13-Pada13) -> 5V_PERM
- J4 pad a14: unconnected-(J4-Pin_a14-Pada14) -> 3.3V
- J4 pad a15: unconnected-(J4-Pin_a15-Pada15) -> GND
- J4 pad a16: unconnected-(J4-Pin_a16-Pada16) -> GND
- J4 pad a2: unconnected-(J4-Pin_a2-Pada2) -> SUN_SENSE_3
- J4 pad a22: unconnected-(J4-Pin_a22-Pada22) -> SOL_PIN
- J4 pad a23: unconnected-(J4-Pin_a23-Pada23) -> BATT_PIN
- J4 pad a24: unconnected-(J4-Pin_a24-Pada24) -> BATT_PIN
- J4 pad a25: unconnected-(J4-Pin_a25-Pada25) -> RBF_A
- J4 pad a26: GND -> DS_A
- J4 pad a3: unconnected-(J4-Pin_a3-Pada3) -> THR_1
- J4 pad a4: unconnected-(J4-Pin_a4-Pada4) -> THR_3
- J4 pad b1: unconnected-(J4-Pin_b1-Padb1) -> SUN_SENSE_2
- J4 pad b10: unconnected-(J4-Pin_b10-Padb10) -> HEATER_PWM
- J4 pad b12: unconnected-(J4-Pin_b12-Padb12) -> 12V
- J4 pad b13: unconnected-(J4-Pin_b13-Padb13) -> 5V_PERM
- J4 pad b14: unconnected-(J4-Pin_b14-Padb14) -> 3.3V
- J4 pad b15: unconnected-(J4-Pin_b15-Padb15) -> GND
- J4 pad b16: unconnected-(J4-Pin_b16-Padb16) -> GND
- J4 pad b2: unconnected-(J4-Pin_b2-Padb2) -> SUN_SENSE_4
- J4 pad b22: unconnected-(J4-Pin_b22-Padb22) -> SOL_PIN
- J4 pad b23: unconnected-(J4-Pin_b23-Padb23) -> SYS_PIN
- J4 pad b24: unconnected-(J4-Pin_b24-Padb24) -> SYS_PIN
- J4 pad b25: unconnected-(J4-Pin_b25-Padb25) -> RBF_B
- J4 pad b26: unconnected-(J4-Pin_b26-Padb26) -> DS_B
- J4 pad b3: unconnected-(J4-Pin_b3-Padb3) -> THR_2
- J4 pad b4: unconnected-(J4-Pin_b4-Padb4) -> THR_4
- J4 pad b5: unconnected-(J4-Pin_b5-Padb5) -> THR_5
- J4 pad b6: unconnected-(J4-Pin_b6-Padb6) -> THR_6
- J4 pad b7: unconnected-(J4-Pin_b7-Padb7) -> THR_7
- J4 pad b8: unconnected-(J4-Pin_b8-Padb8) -> THR_8
- J4 pad b9: unconnected-(J4-Pin_b9-Padb9) -> THR_9
