File: EPS PCB/EPS_PCB_PrototypingV2/.history/EPS_PCB_Prototyping.kicad_pcb (KiCad board)
At the start: 2 copper layers, 95.9 x 90.2 mm, 94 parts, among them J1 Conn_02x26_Row_Letter_First, J2 Conn_02x26_Row_Letter_First, J3 Conn_01x08_Pin, J4 Conn_01x06_Pin, J5 Conn_01x02_Pin, J6 Conn_01x02_Pin, J7 Conn_01x02_Pin, J8 Conn_01x02_Pin, J9 Conn_01x02_Pin, Q1 DMG6968U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

Commit message: PDS Ordered
Parts:
- added J10: Conn_01x02_Pin, Connector_PinSocket_2.54mm:PinSocket_1x02_P2.54mm_Vertical, F.Cu at (215.7, 67.0)
- added J11: Conn_01x02_Pin, Connector_PinSocket_2.54mm:PinSocket_1x02_P2.54mm_Vertical, F.Cu at (215.4, 96.3)
- added J12: Conn_01x02_Pin, Connector_PinSocket_2.54mm:PinSocket_1x02_P2.54mm_Vertical, F.Cu at (210.4, 132.2)
- added J13: Conn_01x02_Pin, Connector_PinSocket_2.54mm:PinSocket_1x02_P2.54mm_Vertical, F.Cu at (189.4, 65.5)
- added J14: Conn_01x02_Pin, Connector_PinSocket_2.54mm:PinSocket_1x02_P2.54mm_Vertical, F.Cu at (189.7, 75.7)
- added J15: Conn_01x02_Pin, Connector_PinSocket_2.54mm:PinSocket_1x02_P2.54mm_Vertical, F.Cu at (192.9, 118.5)
- Q1, Q2, Q5: value DMG6968U -> DMG2305UX
- moved C15 0.77 mm to (191.9, 113.4)
- moved L2 0.45 mm to (209.9, 89.5)
Connections:
- C1 pad 1: V_Batt -> Net-(J10-Pin_2)
- C16 pad 1: 5V_conv_out -> Net-(J13-Pin_2)
- C19 pad 1: 3V3_conv_out -> Net-(J15-Pin_2)
- C2 pad 1: V_Batt -> Net-(J11-Pin_2)
- C26 pad 1: 12V_conv_out -> Net-(J14-Pin_1)
- C3 pad 1: V_Batt -> Net-(J12-Pin_2)
- J1 pad b12: RS-485 SYS1 B -> RS-485 SYS1 A
- U1 pad 7: V_Batt -> Net-(J10-Pin_2)
- U2 pad 7: V_Batt -> Net-(J11-Pin_2)
- U3 pad 7: V_Batt -> Net-(J12-Pin_2)
- U6 pad 11: 3V3_conv_out -> Net-(J15-Pin_2)
- U7 pad 10: 12V_conv_out -> Net-(J14-Pin_1)
- U7 pad 4: 5V_conv_out -> Net-(J13-Pin_2)
Routing:
- net V_Batt: track 217.5 -> 169.4 mm, vias 9 -> 7
- net Net-(J10-Pin_2): track 0.00 -> 16.1 mm, vias 0 -> 1
- net GND: track 158.1 -> 171.8 mm, vias 36 -> 47
- net Net-(J11-Pin_2): track 0.00 -> 12.3 mm
- net Net-(J12-Pin_2): track 0.00 -> 9.71 mm
- net Net-(J15-Pin_2): track 0.00 -> 8.03 mm
- net 3V3_conv_out: track 115.3 -> 111.2 mm, vias 3 -> 1
- net RS-485 SYS1 B: track 2.54 -> 0.00 mm
- net 12V_conv_out: track 26.9 -> 29.1 mm
- net 5V_conv_out: track 10.8 -> 8.78 mm
- net Net-(J13-Pin_2): track 0.00 -> 2.06 mm
- net Net-(J14-Pin_1): track 0.00 -> 1.99 mm
- net 5V_HK: track 273.5 -> 274.3 mm
- added copper zone on F.Cu, net Net-(J13-Pin_2)
- added copper zone on F.Cu, net Net-(J14-Pin_1)
