File: EPS PCB/EPS_PCB_PrototypingV2/.history/curr_meas.kicad_sch (KiCad schematic)
At the start: 36 parts, among them Q1 DMG6968U, Q2 DMG6968U, Q3 2N7002, Q4 2N7002, Q5 DMG6968U, Q6 2N7002, U6 STEF033APUR, U7 STEF512PUR, U8 INA3221

Commit message: PDS Ordered
Parts:
- added J13, J14, J15: Conn_01x02_Pin, Connector_PinSocket_2.54mm:PinSocket_1x02_P2.54mm_Vertical, symbol Connector:Conn_01x02_Pin
- Q1, Q2, Q5: value DMG6968U -> DMG2305UX
Connections:
- net 12V_conv_out: now also J14.2 (Pin_2); no longer C26.1, U7.10 (VIN_12)
- net 3V3_conv_out: now also J15.1 (Pin_1); no longer C19.1, U6.11 (EPAD)
- net 5V_conv_out: now also J13.1 (Pin_1); no longer C16.1, U7.4 (VIN_5)
- new net: C16.1, J13.2 (Pin_2), U7.4 (VIN_5)
- new net: C26.1, J14.1 (Pin_1), U7.10 (VIN_12)
- new net: C19.1, J15.2 (Pin_2), U6.11 (EPAD)
