File: EPS PCB/EPS_PCB_PrototypingV2/.history/pwrconv.kicad_sch (KiCad schematic)
At the start: 35 parts, among them J5 Conn_01x02_Pin, J6 Conn_01x02_Pin, J7 Conn_01x02_Pin, J8 Conn_01x02_Pin, U1 TPS5430DDA, U2 TPS5430DDA, U3 TPS5430DDA, U4 TPS7A1650DGNR

Commit message: PDS Ordered
Parts:
- added J10, J11, J12: Conn_01x02_Pin, Connector_PinSocket_2.54mm:PinSocket_1x02_P2.54mm_Vertical, symbol Connector:Conn_01x02_Pin
Connections:
- net V_Batt: now also J10.1 (Pin_1), J11.1 (Pin_1), J12.1 (Pin_1); no longer C1.1, C2.1, C3.1, U1.7 (VIN), U2.7 (VIN), U3.7 (VIN)
- new net: C3.1, J12.2 (Pin_2), U3.7 (VIN)
- new net: C2.1, J11.2 (Pin_2), U2.7 (VIN)
- new net: C1.1, J10.2 (Pin_2), U1.7 (VIN)
